Commit message: Gazebo simulation launch file for piezo AUV. This launch file sets up the Gazebo environment, spawns the AUV model, and initializes necessary ROS nodes for simulation.

File: piezo_auv_description/urdf/Centroid_body.urdf.xacro (robot description, xacro)
@@ -4,4 +4,11 @@
      For more information, please see http://wiki.ros.org/sw_urdf_exporter -->
 <robot name="Centroid_body" xmlns:xacro="http://www.ros.org/wiki/xacro">
+  <!-- Dummy root link to prevent KDL inertia warning -->
+  <link name="base_footprint"/>
+  <joint name="base_footprint_joint" type="fixed">
+    <parent link="base_footprint"/>
+    <child link="base_link"/>
+    <origin xyz="0 0 0" rpy="0 0 0"/>
+  </joint>
   <link
     name="base_link">
@@ -88,5 +95,5 @@
   </gazebo>
   <joint
-    name="left_jet_f"
+    name="left_jet_f_joint"
     type="fixed">
     <origin
@@ -141,5 +148,5 @@
   </gazebo>
   <joint
-    name="left_jet_r"
+    name="left_jet_r_joint"
     type="fixed">
     <origin
@@ -194,5 +201,5 @@
   </gazebo>
   <joint
-    name="right_jet_f"
+    name="right_jet_f_joint"
     type="fixed">
     <origin
@@ -247,5 +254,5 @@
   </gazebo>
   <joint
-    name="right_jet_r"
+    name="right_jet_r_joint"
     type="fixed">
     <origin
@@ -300,5 +307,5 @@
   </gazebo>
   <joint
-    name="hover_front"
+    name="hover_front_joint"
     type="fixed">
     <origin
@@ -353,5 +360,5 @@
   </gazebo>
   <joint
-    name="hover_rear"
+    name="hover_rear_joint"
     type="fixed">
     <origin

Commit message: Temp

File: piezo_auv_description/urdf/Centroid_body.urdf.xacro (robot description, xacro)
@@ -45,8 +45,7 @@
         xyz="0 0 0"
         rpy="0 0 0" />
-      <geometry>
-        <mesh
-          filename="package://piezo_auv_description/meshes/base_link.STL" />
-      </geometry>
+        <geometry>
+          <box size="0.10964625 0.11001523 0.07"/>
+        </geometry>
     </collision>
   </link>
@@ -372,3 +371,24 @@
       xyz="0 0 0" />
   </joint>
+    <link name="imu_link">
+    <inertial>
+      <mass value="0.001"/>
+      <origin xyz="0 0 0" rpy="0 0 0"/>
+      <inertia ixx="1e-7" iyy="1e-7" izz="1e-7" ixy="0" ixz="0" iyz="0"/>
+    </inertial>
+  </link>
+  <joint name="imu_joint" type="fixed">
+    <origin xyz="0 0 0.005" rpy="0 0 0"/>
+    <parent link="base_link"/>
+    <child link="imu_link"/>
+    <axis xyz="0 0 0"/>
+  </joint>
+  <gazebo reference="imu_link">
+    <sensor name="imu_sensor" type="imu">
+      <always_on>1</always_on>
+      <update_rate>50</update_rate>
+      <visualize>true</visualize>
+      <topic>imu</topic>
+    </sensor>
+  </gazebo>
 </robot>

Commit message: Physics : Complete untill physical tuning

File: piezo_auv_description/urdf/Centroid_body.urdf.xacro (robot description, xacro)
@@ -43,8 +43,8 @@
     <collision>
       <origin
-        xyz="0 0 0"
+        xyz="0 0 0.012"
         rpy="0 0 0" />
         <geometry>
-          <box size="0.10964625 0.11001523 0.07"/>
+          <box size="0.10964625 0.11001523 0.00408" />
         </geometry>
     </collision>
@@ -392,3 +392,33 @@
     </sensor>
   </gazebo>
+    <gazebo>
+      <plugin filename="gz-sim-hydrodynamics-system" name="gz::sim::systems::Hydrodynamics">
+        <link_name>base_footprint</link_name>
+        <xDotU>0.0</xDotU>
+        <yDotV>0.0</yDotV>
+        <zDotW>0.0</zDotW>
+        <kDotP>0.0</kDotP>
+        <mDotQ>0.0</mDotQ>
+        <nDotR>0.0</nDotR>
+        <xU>-0.05</xU>
+        <yV>-0.05</yV>
+        <zW>0.00</zW>
+        <kP>-0.00005</kP>
+        <mQ>-0.00005</mQ>
+        <nR>-0.00005</nR>
+        <xUabsU>-4.24</xUabsU>
+        <yVabsV>-4.22</yVabsV>
+        <zWabsW>-6.63</zWabsW>
+        <kPabsP>-0.00005</kPabsP>
+        <mQabsQ>-0.00005</mQabsQ>
+        <nRabsR>-0.00005</nRabsR>
+      </plugin>
+    </gazebo>
+    <gazebo>
+      <plugin filename="gz-sim-odometry-publisher-system" name="gz::sim::systems::OdometryPublisher">
+        <odom_frame>odom</odom_frame>
+        <robot_base_frame>base_footprint</robot_base_frame>
+        <dimensions>3</dimensions>
+      </plugin>
+    </gazebo>
 </robot>

Commit message: Signal generation redone

File: piezo_auv_description/urdf/Centroid_body.urdf.xacro (robot description, xacro)
@@ -46,5 +46,5 @@
         rpy="0 0 0" />
         <geometry>
-          <box size="0.10964625 0.11001523 0.00408" />
+          <box size="0.10964625 0.11001523 0.0040815" />
         </geometry>
     </collision>
@@ -401,16 +401,18 @@
         <mDotQ>0.0</mDotQ>
         <nDotR>0.0</nDotR>
-        <xU>-0.05</xU>
-        <yV>-0.05</yV>
-        <zW>0.00</zW>
-        <kP>-0.00005</kP>
-        <mQ>-0.00005</mQ>
-        <nR>-0.00005</nR>
-        <xUabsU>-4.24</xUabsU>
-        <yVabsV>-4.22</yVabsV>
-        <zWabsW>-6.63</zWabsW>
-        <kPabsP>-0.00005</kPabsP>
-        <mQabsQ>-0.00005</mQabsQ>
-        <nRabsR>-0.00005</nRabsR>
+        <!-- Realistic Linear Drag (Viscous Skin Friction) -->
+        <xU>-0.15</xU>
+        <yV>-0.15</yV>
+        <zW>-0.20</zW>
+        <kP>-0.001</kP>
+        <mQ>-0.001</mQ>
+        <nR>-0.002</nR>
+        <!-- Realistic Quadratic Form Drag (Re ~ 5,270) -->
+        <xUabsU>-2.95</xUabsU>
+        <yVabsV>-2.95</yVabsV>
+        <zWabsW>-5.28</zWabsW>
+        <kPabsP>-0.0045</kPabsP>
+        <mQabsQ>-0.0045</mQabsQ>
+        <nRabsR>-0.0041</nRabsR>
       </plugin>
     </gazebo>
